File: boards/CP-Sapling/CP Sapling.sch (EAGLE design)
At the start: 17 parts, among them J1 1981568-1, J4 QWIIC_RIGHT_ANGLE, U1 ATSAMD21E18A-AUTTQFP32_MC_MCH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, U2 TLV75533PDBVRDBV5_TEX-L, U3 AT25DF081A-SSH-T

Commit message: Add files via upload
updating board and schematic files
Parts:
- removed LOGO1: QWIIC_LOGO_3MM, SparkFun-Aesthetics:QWIIC_LOGO_3MM
- added TP1, TP2: TEST-POINT3X4, SparkFun-Connectors:TEST-POINT3X4
Connections:
- net D1 renamed NP
- removed net SWCLK/D10: J3.2, U1.PA30
- removed net SWDIO/D12: J3.3, U1.PA31
- new net D10: J3.2, U1.PA00
- new net D11: J3.3, U1.PA01
- new net SWCLK: TP2.1, U1.PA30
- new net SWDIO: TP1.1, U1.PA31
- net DM: now also U1.PA24; no longer U1.PA23
- net DP: now also U1.PA25; no longer U1.PA24
Changed lines of the file:
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@@
 <part name="D1" library="SparkFun-LED" deviceset="WS2812B" device="WS2812B-3535" value="WS2812B"/>
 <part name="J4" library="SparkFun-Connectors" deviceset="QWIIC_CONNECTOR" device="JS-1MM" value="QWIIC_RIGHT_ANGLE"/>
-<part name="LOGO1" library="SparkFun-Aesthetics" deviceset="QWIIC_LOGO" device="_3MM"/>
 <part name="U3" library="AT25DF081A-SSH-T" deviceset="AT25DF081A-SSH-T" device=""/>
+<part name="TP1" library="SparkFun-Connectors" deviceset="TEST-POINT" device="3X4"/>
+<part name="TP2" library="SparkFun-Connectors" deviceset="TEST-POINT" device="3X4"/>
 </parts>
 <sheets>
@@
 <attribute name="NAME" x="14.986" y="12.7" size="1.778" layer="95" font="vector" rot="R90"/>
 </instance>
-<instance part="LOGO1" gate="G$1" x="20.32" y="7.62" smashed="yes"/>
 <instance part="U3" gate="A" x="99.06" y="121.92" smashed="yes">
 <attribute name="NAME" x="119.7356" y="131.0386" size="2.0828" layer="95" ratio="6" rot="SR0"/>
 <attribute name="VALUE" x="119.1006" y="128.4986" size="2.0828" layer="96" ratio="6" rot="SR0"/>
+</instance>
+<instance part="TP1" gate="G$1" x="86.36" y="17.78" smashed="yes" rot="R270">
+<attribute name="NAME" x="88.9" y="20.32" size="1.778" layer="95" font="vector" rot="R270"/>
+<attribute name="VALUE" x="83.82" y="20.32" size="1.778" layer="96" font="vector" rot="R270"/>
+</instance>
+<instance part="TP2" gate="G$1" x="91.44" y="17.78" smashed="yes" rot="R270">
+<attribute name="NAME" x="93.98" y="20.32" size="1.778" layer="95" font="vector" rot="R270"/>
+<attribute name="VALUE" x="88.9" y="20.32" size="1.778" layer="96" font="vector" rot="R270"/>
 </instance>
 </instances>
@@
 </segment>
 <segment>
-<pinref part="U1" gate="A" pin="PA23"/>
-<wire x1="119.38" y1="58.42" x2="121.92" y2="58.42" width="0.1524" layer="91"/>
-<label x="121.92" y="58.42" size="1.778" layer="95" xref="yes"/>
+<pinref part="U1" gate="A" pin="PA24"/>
+<wire x1="119.38" y1="60.96" x2="121.92" y2="60.96" width="0.1524" layer="91"/>
+<label x="121.92" y="60.96" size="1.778" layer="95" xref="yes"/>
 </segment>
 </net>
@@
 </segment>
 <segment>
-<pinref part="U1" gate="A" pin="PA24"/>
-<wire x1="119.38" y1="60.96" x2="121.92" y2="60.96" width="0.1524" layer="91"/>
-<label x="121.92" y="60.96" size="1.778" layer="95" xref="yes"/>
+<pinref part="U1" gate="A" pin="PA25"/>
+<wire x1="119.38" y1="63.5" x2="121.92" y2="63.5" width="0.1524" layer="91"/>
+<label x="121.92" y="63.5" size="1.778" layer="95" xref="yes"/>
 </segment>
 </net>
@@
 </segment>
 </net>
-<net name="SWDIO/D12" class="0">
+<net name="SWDIO" class="0">
 <segment>
 <pinref part="U1" gate="A" pin="PA31"/>
@@
 </segment>
 <segment>
-<wire x1="71.12" y1="22.86" x2="71.12" y2="25.4" width="0.1524" layer="91"/>
-<pinref part="J3" gate="G$1" pin="3"/>
-<label x="71.12" y="25.4" size="1.778" layer="95" rot="R90" xref="yes"/>
-</segment>
-</net>
-<net name="SWCLK/D10" class="0">
+<pinref part="TP1" gate="G$1" pin="1"/>
+<wire x1="86.36" y1="17.78" x2="86.36" y2="20.32" width="0.1524" layer="91"/>
+<label x="86.36" y="20.32" size="1.778" layer="95" rot="R90" xref="yes"/>
+</segment>
+</net>
+<net name="SWCLK" class="0">
 <segment>
 <pinref part="U1" gate="A" pin="PA30"/>
@@
 </segment>
 <segment>
-<wire x1="73.66" y1="22.86" x2="73.66" y2="25.4" width="0.1524" layer="91"/>
-<pinref part="J3" gate="G$1" pin="2"/>
-<label x="73.66" y="25.4" size="1.778" layer="95" rot="R90" xref="yes"/>
+<pinref part="TP2" gate="G$1" pin="1"/>
+<wire x1="91.44" y1="17.78" x2="91.44" y2="20.32" width="0.1524" layer="91"/>
+<label x="91.44" y="20.32" size="1.778" layer="95" rot="R90" xref="yes"/>
 </segment>
 </net>
@@
 </segment>
 </net>
-<net name="D1" class="0">
+<net name="NP" class="0">
 <segment>
 <pinref part="D1" gate="G$1" pin="DI"/>
@@
 </segment>
 </net>
+<net name="D10" class="0">
+<segment>
+<pinref part="U1" gate="A" pin="PA00"/>
+<wire x1="73.66" y1="83.82" x2="71.12" y2="83.82" width="0.1524" layer="91"/>
+<label x="71.12" y="83.82" size="1.778" layer="95" rot="R180" xref="yes"/>
+</segment>
+<segment>
+<wire x1="73.66" y1="22.86" x2="73.66" y2="25.4" width="0.1524" layer="91"/>
+<pinref part="J3" gate="G$1" pin="2"/>
+<label x="73.66" y="25.4" size="1.778" layer="95" rot="R90" xref="yes"/>
+</segment>
+</net>
+<net name="D11" class="0">
+<segment>
+<pinref part="U1" gate="A" pin="PA01"/>
+<wire x1="73.66" y1="81.28" x2="71.12" y2="81.28" width="0.1524" layer="91"/>
+<label x="71.12" y="81.28" size="1.778" layer="95" rot="R180" xref="yes"/>
+</segment>
+<segment>
+<wire x1="71.12" y1="22.86" x2="71.12" y2="25.4" width="0.1524" layer="91"/>
+<pinref part="J3" gate="G$1" pin="3"/>
+<label x="71.12" y="25.4" size="1.778" layer="95" rot="R90" xref="yes"/>
+</segment>
+</net>
