File: boards/PixelWing-ESP32/PixelWing_rev0.1.sch (EAGLE design)
At the start: 70 parts, among them J1 QWIIC_RIGHT_ANGLE, U1 ESP32-S2-WROVER, U2 TLV75533PDBVRDBV5_TEX-L

Commit message: Add files via upload
Other:
- note added: "1.0"
- note added: "Oak Development Technologies By Seth Kerr"
- moved on the sheet: BOOT, C1, C2, C3, C4, C5, D1, D10, D11, D12, D13, D14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
